File: Proyecto/Poncho_Mediano.sch (KiCad schematic (older format))
At the start: 7 parts, among them P1 CONN_5, P2 CONN_4

Commit message: Actualización de documentación y esquemáticos.
Se actualizaron los archivos de datos y caracteristicas de los displays
y se adelantó a un 90% el diseño de los esquemáticos de KiCad.
Parts:
- H1, H2, H3, H4: footprint Poncho_Modelos:Led_Hole -> FootPrints:Led_Hole
Changed lines of the file:
@@
 EESchema Schematic File Version 2
-LIBS:Poncho_Mediano-cache
+LIBS:power
+LIBS:device
+LIBS:transistors
+LIBS:conn
+LIBS:linear
+LIBS:regul
+LIBS:74xx
+LIBS:cmos4000
+LIBS:adc-dac
+LIBS:memory
+LIBS:xilinx
+LIBS:microcontrollers
+LIBS:dsp
+LIBS:microchip
+LIBS:analog_switches
+LIBS:motorola
+LIBS:texas
+LIBS:intel
+LIBS:audio
+LIBS:interface
+LIBS:digital-audio
+LIBS:philips
+LIBS:display
+LIBS:cypress
+LIBS:siliconi
+LIBS:opto
+LIBS:atmel
+LIBS:contrib
+LIBS:valves
 EELAYER 25 0
 EELAYER END
@@
 F 0 "H1" H 7500 6050 60  0000 C CNN
 F 1 "PCB_HOLE" H 7600 5800 60  0000 C CNN
-F 2 "Poncho_Modelos:Led_Hole" H 7400 5950 60  0001 C CNN
+F 2 "FootPrints:Led_Hole" H 7400 5950 60  0001 C CNN
 F 3 "PCB HOLE" H 7500 6050 60  0001 C CNN
 	1    7550 5900
@@
 F 0 "H2" H 8050 6050 60  0000 C CNN
 F 1 "PCB_HOLE" H 8150 5800 60  0000 C CNN
-F 2 "Poncho_Modelos:Led_Hole" H 7950 5950 60  0001 C CNN
+F 2 "FootPrints:Led_Hole" H 7950 5950 60  0001 C CNN
 F 3 "PCB HOLE" H 8050 6050 60  0001 C CNN
 	1    8100 5900
@@
 F 0 "H3" H 8550 6050 60  0000 C CNN
 F 1 "PCB_HOLE" H 8650 5800 60  0000 C CNN
-F 2 "Poncho_Modelos:Led_Hole" H 8450 5950 60  0001 C CNN
+F 2 "FootPrints:Led_Hole" H 8450 5950 60  0001 C CNN
 F 3 "PCB HOLE" H 8550 6050 60  0001 C CNN
 	1    8600 5900
@@
 F 0 "H4" H 9050 6050 60  0000 C CNN
 F 1 "PCB_HOLE" H 9150 5800 60  0000 C CNN
-F 2 "Poncho_Modelos:Led_Hole" H 8950 5950 60  0001 C CNN
+F 2 "FootPrints:Led_Hole" H 8950 5950 60  0001 C CNN
 F 3 "PCB HOLE" H 9050 6050 60  0001 C CNN
 	1    9100 5900
